Commit message: IMU debuing on 10inch hoverboard
Updated robot description for a hoverboard with 10inch wheels and IMU.
Added some debug printouts and topics for debug information.

File: description/ros2_control/hoverboard_driver.ros2_control.xacro (robot description, xacro)
@@ -5,9 +5,9 @@
       <hardware>
         <plugin>hoverboard_driver/hoverboard_driver</plugin>
-        <param name="wheel_radius">0.0825</param>
+        <param name="wheel_radius">0.127</param>
         <param name="max_velocity">1.0</param>
-        <param name="device">/dev/serial/by-id/usb-FTDI_Quad_RS232-HS-if01-port0</param>
-        <!--<param name="imu_enabled">true</param>-->
-        <!--<param name="imu0_frame_id">imu0_link</param>-->
+        <param name="device">/dev/serial/by-path/platform-fd500000.pcie-pci-0000:01:00.0-usb-0:1.3:1.0-port0</param>
+        <param name="imu_enabled">true</param>
+        <param name="imu0_frame_id">imu0_link</param>
         <!--<param name="imu1_frame_id">imu1_link</param>-->
         <!--<param name="linear_acceleration_covariance_diagonal">0.00025 0.00025 0.00025</param>-->

File: description/urdf/diffbot_description.urdf.xacro (robot description, xacro)
@@ -5,12 +5,12 @@
   <xacro:property name="PI" value="3.1415926535897931"/>
   <xacro:property name="base_mass" value="0.3" /> <!-- arbitrary value for base mass -->
-  <xacro:property name="base_width" value="0.1" />
-  <xacro:property name="base_length" value="0.1" />
-  <xacro:property name="base_height" value="0.05" />
+  <xacro:property name="base_width" value="0.60" />
+  <xacro:property name="base_length" value="0.19" />
+  <xacro:property name="base_height" value="0.12" />
   <xacro:property name="wheel_mass" value="0.3" /> <!-- arbitrary value for wheel mass -->
-  <xacro:property name="wheel_len" value="0.020" />
-  <xacro:property name="wheel_radius" value="0.015" />
+  <xacro:property name="wheel_len" value="0.052" />
+  <xacro:property name="wheel_radius" value="0.127" />
   <xacro:property name="caster_wheel_mass" value="0.1" /> <!-- arbitrary value for caster wheel mass -->
-  <xacro:property name="caster_wheel_radius" value="0.015" />
+  <xacro:property name="caster_wheel_radius" value="0.10" />
   <xacro:property name="z_offset" value="-${base_height/2}" /> <!-- Space btw top of beam and the each joint -->
   <!-- Base Link -->
@@ -19,5 +19,5 @@
       <origin xyz="0 0 0" rpy="0 0 0"/>
       <geometry>
-        <box size="${base_width} ${base_length} ${base_height}"/>
+        <box size="${base_length} ${base_width} ${base_height}"/>
       </geometry>
     </collision>
@@ -25,5 +25,5 @@
       <origin xyz="0 0 ${base_height/2}" rpy="0 0 0"/>
       <geometry>
-        <box size="${base_width} ${base_length} ${base_height}"/>
+        <box size="${base_length} ${base_width} ${base_height}"/>
       </geometry>
       <material name="orange"/>
@@ -33,7 +33,7 @@
       <mass value="${base_mass}"/>
       <inertia
-        ixx="${base_mass / 12.0 * (base_length*base_length + base_height*base_height)}" ixy="0.0" ixz="0.0"
-        iyy="${base_mass / 12.0 * (base_height*base_height + base_width*base_width)}" iyz="0.0"
-        izz="${base_mass / 12.0 * (base_width*base_width + base_length*base_length)}"/>
+        ixx="${base_mass / 12.0 * (base_width*base_width + base_height*base_height)}" ixy="0.0" ixz="0.0"
+        iyy="${base_mass / 12.0 * (base_height*base_height + base_length*base_length)}" iyz="0.0"
+        izz="${base_mass / 12.0 * (base_length*base_length + base_width*base_width)}"/>
       </inertial>
     </link>
@@ -158,4 +158,30 @@
         </inertial>
       </link>
+    <!-- IMU MPU6500 Link -->
+    <link name="${prefix}imu0_link">
+      <visual>
+        <origin xyz="0 0 0" rpy="0 0 0"/>
+        <geometry>
+          <box size="0.003 0.003 0.001"/>
+        </geometry>
+        <material name="blue"/>
+      </visual>
+      <collision>
+        <origin xyz="0 0 0" rpy="0 0 0"/>
+        <geometry>
+          <box size="0.003 0.003 0.001"/>
+        </geometry>
+      </collision>
+      <inertial>
+        <origin xyz="0 0 0" rpy="0 0 0"/>
+        <mass value="0.01"/>
+        <inertia ixx="1e-6" ixy="0.0" ixz="0.0" iyy="1e-6" iyz="0.0" izz="1e-6"/>
+      </inertial>
+    </link>
+    <joint name="${prefix}imu_joint" type="fixed">
+      <parent link="${prefix}base_link"/>
+      <child link="${prefix}imu0_link"/>
+      <origin xyz="0 0.09 -0.04" rpy="${PI} 0 0"/>
+    </joint>
   </xacro:macro>
 </robot>
